File: rover/rover.kicad_sch (KiCad schematic)
At the start: 9 parts, among them J1 Conn_01x05_Pin, J2 Conn_01x05_Pin, J3 Conn_01x05_Pin, J4 Conn_01x05_Pin, U1 ESP32-WROOM-32, U2 MPU-6500

Commit message: Update PCB
Parts:
- added J5: Conn_01x04_Pin, symbol Connector:Conn_01x04_Pin
Connections:
- net +12V: now also J2.5 (Pin_5)
- net +5V: now also J5.3 (Pin_3)
- net GND: now also J5.2 (Pin_2)
- net MOISTIN: now reaches U1.10 (IO25)
- net MOISTIN: now also J5.4 (Pin_4)
- net MOISTOUT: now reaches U1.6 (IO34)
- net MOISTOUT: now also J5.1 (Pin_1)
