File: Autonomous-Gardening-Rover-v2-master/untitled.kicad_sch (KiCad schematic)
At the start: 21 parts, among them J13 Conn_01x04_Pin, J3 Conn_01x05_Pin, J4 Conn_01x05_Pin, J5 Conn_01x05_Pin, J6 Conn_01x05_Pin, J7 Conn_01x02_Socket, J8 Conn_01x02_Socket, J9 Conn_01x02_Socket, U3 LM1117DTX-3.3/NOPB, U5 ${SIM.PARAMS}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

Commit message: Update
Parts:
- removed J13: Conn_01x04_Pin, symbol Connector:Conn_01x04_Pin
- removed J7, J9: Conn_01x02_Socket, symbol Connector:Conn_01x02_Socket
- added J13: LINEAR ACTUATOR POWER, TerminalBlock_Phoenix:TerminalBlock_Phoenix_MKDS-1,5-2-5.08_1x02_P5.08mm_Horizontal, symbol Connector:Screw_Terminal_01x02
- added J16: UWB POWER, TerminalBlock_Phoenix:TerminalBlock_Phoenix_MKDS-1,5-2-5.08_1x02_P5.08mm_Horizontal, symbol Connector:Screw_Terminal_01x02
- added J17: LINEAR ACTUATOR SIGNAL, TerminalBlock_Phoenix:TerminalBlock_Phoenix_MKDS-1,5-2-5.08_1x02_P5.08mm_Horizontal, symbol Connector:Conn_01x02_Pin
- added J18: UWB SIGNAL, TerminalBlock_Phoenix:TerminalBlock_Phoenix_MKDS-1,5-4-5.08_1x04_P5.08mm_Horizontal, symbol Connector:Conn_01x04_Pin
- added JP3: SolderJumper_2_Open, Jumper:SolderJumper-2_P1.3mm_Open_RoundedPad1.0x1.5mm, symbol Jumper:SolderJumper_2_Open
- added TP11, TP12: TestPoint, TestPoint:TestPoint_Pad_2.5x2.5mm, symbol Connector:TestPoint
- C7, C8: footprint (none) -> Capacitor_SMD:C_0805_2012Metric_Pad1.18x1.45mm_HandSolder
- J3, J4, J5, J6: footprint (none) -> TerminalBlock_Phoenix:TerminalBlock_Phoenix_MKDS-1,5-5-5.08_1x05_P5.08mm_Horizontal
- J8: footprint (none) -> TerminalBlock_Phoenix:TerminalBlock_Phoenix_MKDS-1,5-2-5.08_1x02_P5.08mm_Horizontal
- R12, R13, R16, R17, R18, R19, R20: footprint (none) -> Resistor_SMD:R_0805_2012Metric_Pad1.20x1.40mm_HandSolder
- U3: footprint NDP0003B -> LM1173.3:NDP0003B
- U5, U8, U9: footprint (none) -> LM358P:P8
Connections:
- net +12V: now also J13.1 (Pin_1)
- net +5V: now also C7.1, U3.3 (INPUT)
- net GND: now also J13.2 (Pin_2), J16.2 (Pin_2), TP12.1
- net at C8.1, U3.4 (OUT): now also JP3.1 (A), TP11.1
- new net +3V3: J16.1 (Pin_1), JP3.2 (B)
- new net LINACT+: J17.1 (Pin_1)
- new net LINACT-: J17.2 (Pin_2)
- new net UWBCLK: J18.2 (Pin_2)
- new net UWBCS: J18.4 (Pin_4)
- new net UWBMISO: J18.3 (Pin_3)
- new net UWBMOSI: J18.1 (Pin_1)

Commit message: Update PCB
Parts:
- removed C7: 100uF, Capacitor_SMD:C_0805_2012Metric_Pad1.18x1.45mm_HandSolder, symbol Device:C_Polarized_Small_US
- removed C8: 10uF, Capacitor_SMD:C_0805_2012Metric_Pad1.18x1.45mm_HandSolder, symbol Device:C_Polarized_Small_US
- removed J13: LINEAR ACTUATOR POWER, TerminalBlock_Phoenix:TerminalBlock_Phoenix_MKDS-1,5-2-5.08_1x02_P5.08mm_Horizontal, symbol Connector:Screw_Terminal_01x02
- removed J16: UWB POWER, TerminalBlock_Phoenix:TerminalBlock_Phoenix_MKDS-1,5-2-5.08_1x02_P5.08mm_Horizontal, symbol Connector:Screw_Terminal_01x02
- removed J17: LINEAR ACTUATOR SIGNAL, TerminalBlock_Phoenix:TerminalBlock_Phoenix_MKDS-1,5-2-5.08_1x02_P5.08mm_Horizontal, symbol Connector:Conn_01x02_Pin
- removed J18: UWB SIGNAL, TerminalBlock_Phoenix:TerminalBlock_Phoenix_MKDS-1,5-4-5.08_1x04_P5.08mm_Horizontal, symbol Connector:Conn_01x04_Pin
- removed J3, J4, J5, J6: Conn_01x05_Pin, TerminalBlock_Phoenix:TerminalBlock_Phoenix_MKDS-1,5-5-5.08_1x05_P5.08mm_Horizontal, symbol Connector:Conn_01x05_Pin
- removed J8: Conn_01x02_Socket, TerminalBlock_Phoenix:TerminalBlock_Phoenix_MKDS-1,5-2-5.08_1x02_P5.08mm_Horizontal, symbol Connector:Conn_01x02_Socket
- removed JP3: SolderJumper_2_Open, Jumper:SolderJumper-2_P1.3mm_Open_RoundedPad1.0x1.5mm, symbol Jumper:SolderJumper_2_Open
- removed R12, R13: 100K, Resistor_SMD:R_0805_2012Metric_Pad1.20x1.40mm_HandSolder, symbol Device:R
- removed R16: 10M, Resistor_SMD:R_0805_2012Metric_Pad1.20x1.40mm_HandSolder, symbol Device:R
- removed R17, R18, R19, R20: 1K, Resistor_SMD:R_0805_2012Metric_Pad1.20x1.40mm_HandSolder, symbol Device:R
- removed TP11, TP12: TestPoint, TestPoint:TestPoint_Pad_2.5x2.5mm, symbol Connector:TestPoint
- removed U3: LM1117DTX-3.3/NOPB, LM1173.3:NDP0003B, symbol LM1117:LM1117DTX-3.3_NOPB
- removed U5, U8, U9: ${SIM.PARAMS}, LM358P:P8, symbol Simulation_SPICE:OPAMP
