File: Autonomous-Gardening-Rover-v2-master/Autonomous_Gardening_Rover_v2.kicad_sch (KiCad schematic)
At the start: 48 parts, among them J1 Screw_Terminal_01x02, J10 Conn_01x09_Socket, J11 Conn_01x02_Socket, J12 Conn_01x02_Pin, J2 USB_B_Micro, Q1 BC107, Q2 BC107, Q3 AO4485, SW1 SW_Push, SW2 SW_Push, U1 ESP32-S3-WROOM-1, U2 CP2104, U6 MPU-6500, U7 TPS62933DRLR

Commit message: Update
Parts:
- removed J11: Conn_01x02_Socket, symbol Connector:Conn_01x02_Socket
- removed J12: Conn_01x02_Pin, symbol Connector:Conn_01x02_Pin
- added H1, H2, H3, H4: MountingHole, MountingHole:MountingHole_3.2mm_M3, symbol Mechanical:MountingHole
- added J15: Conn_01x02_Pin, TerminalBlock_Phoenix:TerminalBlock_Phoenix_MKDS-1,5-2-5.08_1x02_P5.08mm_Horizontal, symbol Connector:Conn_01x02_Pin
- added J7: MPU SIGNAL, TerminalBlock_Phoenix:TerminalBlock_Phoenix_MKDS-1,5-5-5.08_1x05_P5.08mm_Horizontal, symbol Connector:Conn_01x05_Pin
- added J9: MPU POWER, TerminalBlock_Phoenix:TerminalBlock_Phoenix_MKDS-1,5-2-5.08_1x02_P5.08mm_Horizontal, symbol Connector:Conn_01x02_Pin
- added JP2: SolderJumper_2_Open, Jumper:SolderJumper-2_P1.3mm_Open_RoundedPad1.0x1.5mm, symbol Jumper:SolderJumper_2_Open
- added TP1, TP10, TP2, TP3, TP4, TP5, TP8: TestPoint, TestPoint:TestPoint_Pad_2.5x2.5mm, symbol Connector:TestPoint
- added TP6: TEST GPIO0_STRAPPING, TestPoint:TestPoint_Pad_2.5x2.5mm, symbol Connector:TestPoint
- added TP7: TEST CHIP_PU, TestPoint:TestPoint_Pad_2.5x2.5mm, symbol Connector:TestPoint
- added TP9: TEST GND, TestPoint:TestPoint_Pad_2.5x2.5mm, symbol Connector:TestPoint
- C1, C15, C16, C17, C18, C19, C2, C20, C21, C22, C3, C4, C5, C6: footprint (none) -> Capacitor_SMD:C_0805_2012Metric_Pad1.18x1.45mm_HandSolder
- D1: footprint (none) -> Diode_SMD:D_SOD-123
- D2, D3: footprint (none) -> Package_TO_SOT_SMD:TSOT-23_HandSoldering
- F1: footprint (none) -> Fuse:Fuseholder_Littelfuse_Nano2_154x
- J1: value Screw_Terminal_01x02 -> 12V BATTERY POWER; footprint (none) -> TerminalBlock_Phoenix:TerminalBlock_Phoenix_MKDS-1,5-2-5.08_1x02_P5.08mm_Horizontal
- J10: value Conn_01x09_Socket -> SENSORS; footprint (none) -> Connector_PinHeader_2.54mm:PinHeader_1x09_P2.54mm_Vertical
- J2: footprint (none) -> Connector_USB:USB_Micro-B_Molex_47346-0001
- JP1: footprint (none) -> Jumper:SolderJumper-2_P1.3mm_Open_RoundedPad1.0x1.5mm
- L2: footprint (none) -> Inductor_Custom:Inductor_Custom
- Q3: footprint local_footprints:SO8SOP-8L_AOS -> AO4485:SO8SOP-8L_AOS
- R1, R10, R11, R14, R15, R2, R3, R4, R5, R6, R7, R8, R9: footprint (none) -> Resistor_SMD:R_0805_2012Metric_Pad1.20x1.40mm_HandSolder
- SW1, SW2: footprint (none) -> Button_Switch_SMD:SW_DIP_SPSTx01_Slide_Copal_CHS-01A_W5.08mm_P1.27mm_JPin
- U6: footprint QFN24_3X3X0P9_IVS -> MPU6500:QFN24_3X3X0P9_IVS
- U7: footprint SOT-5X3-8_DRL_TEX -> TSP62933DRLR:SOT-5X3-8_DRL_TEX
Connections:
- net 3V3 is gone; now on net +3V3: J10.2 (Pin_2), J10.5 (Pin_5)
- net Vin is gone; now on net +12V: C18.1, C19.1, U7.3 (VIN)
- net +3.3V: no longer C1.1, C15.2, C2.1, U1.2 (3V3), U6.8 (VDDIO)
- net +3V3: now also C1.1, C15.2, C18.2, C19.2, C2.1, C20.2, J1.1 (Pin_1), U1.2 (3V3), U6.8 (VDDIO), J15.2 (Pin_2), J9.2 (Pin_2), TP10.1, TP5.1, TP9.1
- net +5V: now also J9.1 (Pin_1), JP2.2 (B)
- net CHIP_PU: now also TP7.1
- net D+: now also TP3.1
- net D-: now also TP4.1
- net DTR: now also TP1.1
- net GPIO0_STRAPPING: now also TP6.1
- net GPIO3_STRAPPING: now also R3.2
- net MPUCLK: now also J7.2 (Pin_2)
- net MPUCS: now also J7.4 (Pin_4)
- net MPUINT: now also J7.5 (Pin_5)
- net MPUMISO: now also J7.3 (Pin_3)
- net MPUMOSI: now also J7.1 (Pin_1)
- net RTS: now also TP2.1
- net VBAT_READ: now also J15.1 (Pin_1)
- net at C22.1, L2.2, R14.1: now also JP2.1 (A), TP8.1
- net at F1.1: now also J1.2 (Pin_2)
- net UWBCS: now reaches U1.17 (IO9)
- net LINACT-: now reaches U1.18 (IO10)
- net UWBMOSI: now reaches U1.28 (IO35)
- net UWBCLK: now reaches U1.29 (IO36)
- net UWBMISO: now reaches U1.30 (IO37)
- net MOTOR3PWM: now reaches U1.32 (IO39)
- net MOTOR3FG: now reaches U1.33 (IO40)
- net MOTOR4PWM: now reaches U1.34 (IO41)
- net MOTOR4FG: now reaches U1.35 (IO42)
- net +BATT renamed +12V
- net LINEARACT renamed LINACT+
Other:
- moved on the sheet: J1

Commit message: Update PCB
Parts:
- removed C18: 10uF, Capacitor_SMD:C_0805_2012Metric_Pad1.18x1.45mm_HandSolder, symbol Device:C_Small
- removed C19, C21: 100nF, Capacitor_SMD:C_0805_2012Metric_Pad1.18x1.45mm_HandSolder, symbol Device:C_Small
- removed C20: 33nF, Capacitor_SMD:C_0805_2012Metric_Pad1.18x1.45mm_HandSolder, symbol Device:C_Small
- removed C22: 47u, Capacitor_SMD:C_0805_2012Metric_Pad1.18x1.45mm_HandSolder, symbol Device:C_Small
- removed D1: D_Zener, Diode_SMD:D_SOD-123, symbol Device:D_Zener
- removed D2, D3: D_Schottky, Package_TO_SOT_SMD:TSOT-23_HandSoldering, symbol Device:D_Schottky
- removed F1: Fuse, Fuse:Fuseholder_Littelfuse_Nano2_154x, symbol Device:Fuse
- removed J1: 12V BATTERY POWER, TerminalBlock_Phoenix:TerminalBlock_Phoenix_MKDS-1,5-2-5.08_1x02_P5.08mm_Horizontal, symbol Connector:Screw_Terminal_01x02
- removed J15: Conn_01x02_Pin, TerminalBlock_Phoenix:TerminalBlock_Phoenix_MKDS-1,5-2-5.08_1x02_P5.08mm_Horizontal, symbol Connector:Conn_01x02_Pin
- removed J9: MPU POWER, TerminalBlock_Phoenix:TerminalBlock_Phoenix_MKDS-1,5-2-5.08_1x02_P5.08mm_Horizontal, symbol Connector:Conn_01x02_Pin
- removed JP1, JP2: SolderJumper_2_Open, Jumper:SolderJumper-2_P1.3mm_Open_RoundedPad1.0x1.5mm, symbol Jumper:SolderJumper_2_Open
- removed L2: 7.8uH, Inductor_Custom:Inductor_Custom, symbol Device:L
- removed Q3: AO4485, AO4485:SO8SOP-8L_AOS, symbol local_symbols:AO4485
- removed R10, R9: 100k, Resistor_SMD:R_0805_2012Metric_Pad1.20x1.40mm_HandSolder, symbol Device:R
- removed R11, R15: 10k, Resistor_SMD:R_0805_2012Metric_Pad1.20x1.40mm_HandSolder, symbol Device:R
- removed R14: 52.3k, Resistor_SMD:R_0805_2012Metric_Pad1.20x1.40mm_HandSolder, symbol Device:R
- removed R3: 1k, Resistor_SMD:R_0805_2012Metric_Pad1.20x1.40mm_HandSolder, symbol Device:R
- removed TP10, TP8: TestPoint, TestPoint:TestPoint_Pad_2.5x2.5mm, symbol Connector:TestPoint
- removed U7: TPS62933DRLR, TSP62933DRLR:SOT-5X3-8_DRL_TEX, symbol TPS62933DRLR:TPS62933DRLR
- added J1, J12, J14, J3: Conn_01x05_Pin, TerminalBlock_Phoenix:TerminalBlock_Phoenix_MKDS-1,5-5-5.08_1x05_P5.08mm_Horizontal, symbol Connector:Conn_01x05_Pin
- added J11: Conn_01x02_Socket, TerminalBlock_Phoenix:TerminalBlock_Phoenix_MKDS-1,5-2-5.08_1x02_P5.08mm_Horizontal, symbol Connector:Conn_01x02_Socket
- added J24: UWB SIGNAL, TerminalBlock_Phoenix:TerminalBlock_Phoenix_MKDS-1,5-4-5.08_1x04_P5.08mm_Horizontal, symbol Connector:Conn_01x04_Pin
- added J4: LINEAR ACTUATOR SIGNAL, TerminalBlock_Phoenix:TerminalBlock_Phoenix_MKDS-1,5-2-5.08_1x02_P5.08mm_Horizontal, symbol Connector:Conn_01x02_Pin
- added J5, J6, J8: Screw_Terminal_01x02, TerminalBlock_Phoenix:TerminalBlock_Phoenix_MKDS-1,5-2-5.08_1x02_P5.08mm_Horizontal, symbol Connector:Screw_Terminal_01x02
- added JP1: SolderJumper_3_Open, Jumper:SolderJumper-3_P2.0mm_Open_TrianglePad1.0x1.5mm, symbol Jumper:SolderJumper_3_Open
- added R21, R22: 100K, Resistor_SMD:R_0805_2012Metric_Pad1.20x1.40mm_HandSolder, symbol Device:R
- added R23: 10M, Resistor_SMD:R_0805_2012Metric_Pad1.20x1.40mm_HandSolder, symbol Device:R
- added R24, R25, R26, R27: 1K, Resistor_SMD:R_0805_2012Metric_Pad1.20x1.40mm_HandSolder, symbol Device:R
- added R3: 1k, Resistor_SMD:R_0805_2012Metric, symbol basic:R
- added U3, U4: LM358, LM358P:P8, symbol Amplifier_Operational:LM358
- SW1, SW2: footprint Button_Switch_SMD:SW_DIP_SPSTx01_Slide_Copal_CHS-01A_W5.08mm_P1.27mm_JPin -> Button_Switch_THT:SW_PUSH_6mm_H5mm
Connections:
- net +3.3V is gone; now on net +3V3: C17.1, U6.13 (VDD)
- net +12V: now also J1.5 (Pin_5), J12.5 (Pin_5), J14.5 (Pin_5), J3.5 (Pin_5), J5.2 (Pin_2)
- net +3V3: now also J8.2 (Pin_2), JP1.3 (B), R21.2, U3.3 (+), U3.8 (V+), U4.8 (V+); no longer C1.2, C15.1, C16.1, C17.2, C2.2, C3.2, C4.2, C5.2, C6.2, D4.1 (A), J10.3 (Pin_3), J10.6 (Pin_6), J2.5 (GND), SW1.1, SW2.1, TP5.1, TP9.1, U1.1 (GND), U1.40 (GND), U1.41 (GND), U2.2 (GND), U2.25 (GND), U6.18 (GND)
- net +5V: now also J1.3 (Pin_3), J12.3 (Pin_3), J14.3 (Pin_3), J3.3 (Pin_3), J6.2 (Pin_2)
- net GPIO3_STRAPPING: now also R3.1
- net LINACT+: now also J4.1 (Pin_1)
- net LINACT-: now also J4.2 (Pin_2)
- net MOTOR1FG: now also J12.4 (Pin_4)
- net MOTOR1PWM: now also J12.1 (Pin_1)
- net MOTOR2FG: now also J14.4 (Pin_4)
- net MOTOR2PWM: now also J14.1 (Pin_1)
- net MOTOR3FG: now also J1.4 (Pin_4)
- net MOTOR3PWM: now also J1.1 (Pin_1)
- net MOTOR4FG: now also J3.4 (Pin_4)
- net MOTOR4PWM: now also J3.1 (Pin_1)
- net Moisture_Sensor_Output: now also R27.2, U4.1
- net UWBCLK: now also J24.2 (Pin_2)
- net UWBCS: now also J24.4 (Pin_4)
- net UWBMISO: now also J24.3 (Pin_3)
- net UWBMOSI: now also J24.1 (Pin_1)
- new net: R25.2, R27.1, U4.2 (-)
- new net: R24.2, R26.2, U4.3 (+)
- new net: R22.2, R23.2, U3.5 (+)
- new net: R25.1, U3.6 (-), U3.7
- new net: R24.1, U3.1, U3.2 (-)
- new net: JP1.2 (C), R3.2
- new net GND: C1.2, C15.1, C16.1, C17.2, C2.2, C3.2, C4.2, C5.2, C6.2, D4.1 (A), J1.2 (Pin_2), J10.3 (Pin_3), J10.6 (Pin_6), J12.2 (Pin_2), J14.2 (Pin_2), J2.5 (GND), J3.2 (Pin_2), J5.1 (Pin_1), J6.1 (Pin_1), J8.1 (Pin_1), JP1.1 (A), R23.1, R26.1, SW1.1, SW2.1, TP5.1, TP9.1, U1.1 (GND), U1.40 (GND), U1.41 (GND), U2.2 (GND), U2.25 (GND), U3.4 (V-), U4.4 (V-), U6.18 (GND)
- new net Input_Probe_1: J11.1 (Pin_1), R21.1
- new net Input_Probe_2: J11.2 (Pin_2), R22.1
Other:
- moved on the sheet: C5, H1, H2, H3, H4, TP9

Commit message: Update PCB
Parts:
- added R9: 4.7k, Resistor_SMD:R_0805_2012Metric_Pad1.20x1.40mm_HandSolder, symbol Device:R
Connections:
- net +3V3: now also R9.1
- net GND: now also J2.6 (Shield)
- net at U2.9 (~{RST}): now also R9.2
Other:
- moved on the sheet: C6, R4

Commit message: Update PCBS
Parts:
- U1: footprint RF_Module:ESP32-S3-WROOM-1 -> ESP32:ESP32-S3-WROOM-1_EXP
Changed lines of the file:
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@@
 			)
 		)
-		(property "Footprint" "RF_Module:ESP32-S3-WROOM-1"
+		(property "Footprint" "ESP32:ESP32-S3-WROOM-1_EXP"
 			(at 254 66.04 0)
 			(effects
