File: Rover_V5/Autonomous-Gardening-Rover-v2-master/Autonomous_Gardening_Rover_v2.kicad_pcb (KiCad board)
At the start: 2 copper layers, 97.5 x 81.7 mm, 42 parts, among them J10 SENSORS, J11 UWB SIGNALS, J13 MOTOR4SIGNAL, J2 USB_B_Micro, J3 Moisture_Power, J4 LINEAR ACTUATOR SIGNAL, J5 MOTOR1SIGNAL, J6 Screw_Terminal_01x02, J7 MOTOR2SIGNAL, J8 Screw_Terminal_01x02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

Commit message: New version
Routing:
- net GND: track 31.6 -> 35.6 mm, vias 6 -> 9
Changed lines of the file:
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@@
+	)
+	(segment
+		(start 69.25 40.96)
+		(end 69.25 41.25)
+		(width 0.254)
+		(layer "F.Cu")
+		(net 6)
 	)
 	(segment
@@
 		(end 67 64)
 		(width 0.508)
-		(layer "F.Cu")
-		(net 6)
-	)
-	(segment
-		(start 69.25 40.96)
-		(end 69.25 41.25)
-		(width 0.254)
 		(layer "F.Cu")
 		(net 6)
@@
 		(width 0.254)
 		(layer "F.Cu")
+		(net 6)
+	)
+	(via
+		(at 51 38)
+		(size 0.6)
+		(drill 0.3)
+		(layers "F.Cu" "B.Cu")
+		(free yes)
 		(net 6)
 	)
@@
 	)
 	(via
+		(at 68 37.5)
+		(size 0.6)
+		(drill 0.3)
+		(layers "F.Cu" "B.Cu")
+		(free yes)
+		(net 6)
+	)
+	(via
 		(at 51.75 61.25)
 		(size 0.6)
@@
 		(net 6)
 	)
+	(via
+		(at 47 38)
+		(size 0.6)
+		(drill 0.3)
+		(layers "F.Cu" "B.Cu")
+		(free yes)
+		(net 6)
+	)
 	(segment
 		(start 49.5 59)
@@
 		(layer "B.Cu")
 		(net 6)
+	)
+	(segment
+		(start 51 38)
+		(end 47 38)
+		(width 0.2)
+		(layer "B.Cu")
+		(net 6)
