File: power_board_fixed/power_board_fixed/PCB_split/PCB_split.kicad_pcb (KiCad board)
At the start: 2 copper layers, 93 x 93 mm, 40 parts, among them J1 LINEAR ACTUATOR POWER, J10 MOTOR2 POWER, J11 MOTOR3 POWER, J12 MOTOR4 POWER, J13 MOTOR1 EN, J14 MOTOR2 EN, J15 MOTOR3 EN, J16 MOTOR4 EN, J17 LIN REG, J2 LIN ACT DRIVER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

Commit message: New version
Routing:
- net +5V: track 217.8 -> 244.5 mm
- net GND: track 71.8 -> 73.3 mm
Changed lines of the file:
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@@
 		(layer "Edge.Cuts")
-	)
-	(dimension
-		(type aligned)
-		(layer "Edge.Cuts")
-		(pts
-			(xy 181 65) (xy 88 65)
-		)
-		(height 3.499999)
-		(gr_text "93.0000 mm"
-			(at 134.5 60.350001 0)
-			(layer "Edge.Cuts")
-			(effects
-				(font
-					(size 1 1)
-					(thickness 0.15)
-				)
-			)
-		)
-		(format
-			(prefix "")
-			(suffix "")
-			(units 3)
-			(units_format 1)
-			(precision 4)
-		)
-		(style
-			(thickness 0.05)
-			(arrow_length 1.27)
-			(text_position_mode 0)
-			(extension_height 0.58642)
-			(extension_offset 0.5) keep_text_aligned)
-	)
-	(dimension
-		(type aligned)
-		(layer "Edge.Cuts")
-		(pts
-			(xy 181 65) (xy 181 158)
-		)
-		(height 0)
-		(gr_text "93.0000 mm"
-			(at 179.85 111.5 90)
-			(layer "Edge.Cuts")
-			(effects
-				(font
-					(size 1 1)
-					(thickness 0.15)
-				)
-			)
-		)
-		(format
-			(prefix "")
-			(suffix "")
-			(units 3)
-			(units_format 1)
-			(precision 4)
-		)
-		(style
-			(thickness 0.05)
-			(arrow_length 1.27)
-			(text_position_mode 0)
-			(extension_height 0.58642)
-			(extension_offset 0.5) keep_text_aligned)
 	)
 	(segment
@@
 	)
 	(segment
-		(start 101 100)
-		(end 100 100)
+		(start 101.425 100.425)
+		(end 101 100)
 		(width 0.508)
 		(layer "F.Cu")
@@
 	)
 	(segment
+		(start 101.425 126.545)
+		(end 101.425 100.425)
+		(width 0.508)
+		(layer "F.Cu")
+		(net 1)
+	)
+	(segment
 		(start 164.5 128.58)
 		(end 174 138.08)
@@
 	)
 	(segment
+		(start 94.305 126.545)
+		(end 101.425 126.545)
+		(width 0.508)
+		(layer "F.Cu")
+		(net 1)
+	)
+	(segment
 		(start 173.695 93.955)
 		(end 168.045 93.955)
@@
 	)
 	(segment
+		(start 100 100)
+		(end 101 100)
+		(width 0.508)
+		(layer "F.Cu")
+		(net 1)
+	)
+	(segment
 		(start 161.545 93.955)
 		(end 161.5 94)
@@
 		(start 162.65 107.5)
 		(end 162.65 108.91)
-		(width 0.508)
-		(layer "F.Cu")
-		(net 1)
-	)
-	(segment
-		(start 94.305 126.545)
-		(end 101.425 126.545)
 		(width 0.508)
 		(layer "F.Cu")
@@
 	)
 	(segment
-		(start 105.965 94.465)
-		(end 108 96.5)
+		(start 107.465 94.465)
+		(end 94.305 94.465)
 		(width 0.508)
 		(layer "F.Cu")
@@
 	)
 	(segment
-		(start 94.305 94.465)
-		(end 105.965 94.465)
-		(width 0.508)
-		(layer "F.Cu")
-		(net 2)
-	)
-	(segment
 		(start 129.0375 124.0375)
 		(end 124 119)
@@
 	)
 	(segment
+		(start 108 96.5)
+		(end 108 98)
+		(width 0.508)
+		(layer "F.Cu")
+		(net 2)
+	)
+	(segment
+		(start 108 95)
+		(end 107.465 94.465)
+		(width 0.508)
+		(layer "F.Cu")
+		(net 2)
+	)
+	(segment
 		(start 119.5 117.5)
 		(end 122.5 117.5)
@@
 	)
 	(segment
+		(start 108 96.5)
+		(end 108 95)
+		(width 0.508)
+		(layer "F.Cu")
+		(net 2)
+	)
+	(segment
 		(start 109.179 95.321)
 		(end 114.496 95.321)
@@
 		(start 108 96.5)
 		(end 109.179 95.321)
-		(width 0.508)
-		(layer "F.Cu")
-		(net 2)
-	)
-	(segment
-		(start 105.836 98.664)
-		(end 105.836 102.496)
 		(width 0.508)
 		(layer "F.Cu")
@@
 	)
 	(segment
-		(start 108 96.5)
-		(end 105.836 98.664)
+		(start 105.836 99.164)
+		(end 105.836 99.5)
+		(width 0.508)
+		(layer "F.Cu")
+		(net 2)
+	)
+	(segment
+		(start 105.836 99.5)
+		(end 105.836 102.496)
+		(width 0.508)
+		(layer "F.Cu")
+		(net 2)
+	)
+	(segment
+		(start 106.5 98.5)
+		(end 105.836 99.164)
 		(width 0.508)
 		(layer "F.Cu")
@@
 		(width 0.508)
 		(layer "F.Cu")
+		(net 2)
+	)
+	(segment
+		(start 108 98)
+		(end 107.5 98.5)
+		(width 0.508)
+		(layer "F.Cu")
+		(net 2)
+	)
+	(segment
+		(start 107.5 98.5)
+		(end 106.5 98.5)
+		(width 0.508)
+		(layer "F.Cu")
