File: power_board_fixed_regulator/power_board_fixed_regulator/power_board_fixed_regulator.kicad_pcb (KiCad board)
At the start: 2 copper layers, 57 x 30 mm, 14 parts, among them J1 Input, J2 MAIN_BOARD, J3 UWB_POWER, J4 BACK_TO_BUCK, U1 LM1117DTX-3.3/NOPB

Commit message: New version
Parts:
- moved H1 2.06 mm to (63.0, 81.0)
- moved H4 2.06 mm to (63.0, 104.0)
- moved H2 0.71 mm to (114.5, 81.0)
- moved H3 0.71 mm to (114.5, 104.0)
Other:
- board size 57 x 30 mm -> 58.5 x 30 mm
Changed lines of the file:
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@@
 	(footprint "MountingHole:MountingHole_3.2mm_M3"
 		(layer "F.Cu")
-		(at 65 103.5)
+		(at 63 104)
 		(descr "Mounting Hole 3.2mm, no annular, M3")
 		(tags "mounting hole 3.2mm no annular m3")
@@
 	(footprint "MountingHole:MountingHole_3.2mm_M3"
 		(layer "F.Cu")
-		(at 114 81.5)
+		(at 114.5 81)
 		(descr "Mounting Hole 3.2mm, no annular, M3")
 		(tags "mounting hole 3.2mm no annular m3")
@@
 	(footprint "MountingHole:MountingHole_3.2mm_M3"
 		(layer "F.Cu")
-		(at 114 103.5)
+		(at 114.5 104)
 		(descr "Mounting Hole 3.2mm, no annular, M3")
 		(tags "mounting hole 3.2mm no annular m3")
@@
 	(footprint "MountingHole:MountingHole_3.2mm_M3"
 		(layer "F.Cu")
-		(at 65 81.5)
+		(at 63 81)
 		(descr "Mounting Hole 3.2mm, no annular, M3")
 		(tags "mounting hole 3.2mm no annular m3")
@@
 	)
 	(gr_rect
-		(start 61 77.5)
+		(start 59.5 77.5)
 		(end 118 107.5)
 		(stroke
