File: Rover_V7/Autonomous-Gardening-Rover-v2-master/Autonomous_Gardening_Rover_v2.kicad_sch (KiCad schematic)
At the start: 42 parts, among them J10 SENSORS, J11 UWB SIGNALS, J13 MOTOR4SIGNAL, J2 USB_B_Micro, J3 Moisture_Power, J4 LINEAR ACTUATOR SIGNAL, J5 MOTOR1SIGNAL, J6 Screw_Terminal_01x02, J7 MOTOR2SIGNAL, J8 Screw_Terminal_01x02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

Commit message: Add V7
Parts:
- removed J13: MOTOR4SIGNAL, TerminalBlock_Phoenix:TerminalBlock_Phoenix_MKDS-1,5-2-5.08_1x02_P5.08mm_Horizontal, symbol Connector:Conn_01x02_Pin
- removed J5: MOTOR1SIGNAL, TerminalBlock_Phoenix:TerminalBlock_Phoenix_MKDS-1,5-2-5.08_1x02_P5.08mm_Horizontal, symbol Connector:Conn_01x02_Pin
- removed J7: MOTOR2SIGNAL, TerminalBlock_Phoenix:TerminalBlock_Phoenix_MKDS-1,5-2-5.08_1x02_P5.08mm_Horizontal, symbol Connector:Conn_01x02_Pin
- removed J9: MOTOR3SIGNAL, TerminalBlock_Phoenix:TerminalBlock_Phoenix_MKDS-1,5-2-5.08_1x02_P5.08mm_Horizontal, symbol Connector:Conn_01x02_Pin
- removed R10, R11, R12, R13: 5k, Resistor_SMD:R_0805_2012Metric_Pad1.20x1.40mm_HandSolder, symbol Device:R
- removed U1: ESP32-S3-WROOM-1, ESP32:ESP32-S3-WROOM-1_EXP, symbol RF_Module:ESP32-S3-WROOM-1
- added J1: Conn_01x03_Pin, Connector_PinHeader_1.00mm:PinHeader_1x03_P1.00mm_Horizontal, symbol Connector:Conn_01x03_Pin
- added J5, J7, J9: Conn_01x03_Pin, Connector_PinHeader_2.54mm:PinHeader_1x03_P2.54mm_Horizontal, symbol Connector:Conn_01x03_Pin
- added U3: ESP32-S3-WROOM-1-N16R8, ESP32 S3 WROOM 1 N16R8:ESP32-S3-WROOM-1_EXP, symbol 2024-11-21_23-31-15:ESP32-S3-WROOM-1-N16R8
- C2: value 100 uF -> 100 n
Connections:
- net +3V3: now also U3.2 (3V3)
- net CHIP_PU: now also U3.3 (EN)
- net GND: now also U3.1 (GND), U3.40 (GND), U3.41 (GND), U3.46 (GND), U3.47 (GND), U3.48 (GND), U3.49 (GND)
- net GPIO0_STRAPPING: now also U3.27 (IO0)
- net GPIO3_STRAPPING: now also U3.15 (IO3)
- net GPIO46_STRAPPING: now also U3.16 (IO46)
- net LINACT+: now also U3.35 (IO42)
- net LINACT-: now also U3.34 (IO41)
- net MOTOR1PWM: now also J9.1 (Pin_1), U3.31 (IO38)
- net MOTOR2PWM: now also J1.1 (Pin_1), U3.30 (IO37)
- net MOTOR3PWM: now also J5.1 (Pin_1), U3.29 (IO36)
- net MOTOR4PWM: now also J7.1 (Pin_1), U3.28 (IO35)
- net RXD: now also U3.37 (TXD0)
- net TXD: now also U3.36 (RXD0)
- net UWBCLK: now also U3.18 (IO10)
- net UWBCS: now also U3.20 (IO12)
- net UWBINT: now also U3.21 (IO13)
- net UWBMISO: now also U3.19 (IO11)
- net UWBMOSI: now also U3.17 (IO9)
- net pH_Sensor: now also U3.23 (IO21)
- net temp_Sensor: now also U3.24 (IO47)
- new net GPIO1: U3.39 (IO1)
- new net GPIO19: U3.13 (IO19)
- new net GPIO2: U3.38 (IO2)
- new net GPIO20: U3.14 (IO20)
- new net GPIO39: U3.32 (IO39)
- new net GPIO40: U3.33 (IO40)
- new net GPIO45: U3.26 (IO45)
- new net GPIO48: U3.25 (IO48)
- new net GPIO8: U3.12 (IO8)
- new net MOSITURE_SENSOR_OUTPUT: U3.22 (IO14)
- new net MOTOR1ENA: J9.2 (Pin_2), U3.4 (IO4)
- new net MOTOR1ENB: J9.3 (Pin_3), U3.5 (IO5)
- new net MOTOR2ENA: J1.2 (Pin_2), U3.6 (IO6)
- new net MOTOR2ENB: J1.3 (Pin_3), U3.7 (IO7)
- new net MOTOR3ENA: J5.2 (Pin_2), U3.8 (IO15)
- new net MOTOR3ENB: J5.3 (Pin_3), U3.9 (IO16)
- new net MOTOR4ENA: J7.2 (Pin_2), U3.10 (IO17)
- new net MOTOR4ENB: J7.3 (Pin_3), U3.11 (IO18)
Other:
- moved on the sheet: C1, C2, C3, C4, JP1, Q1, Q2, R1, R2, R3, R4, R5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

Commit message: Finish v7 pcb
Parts:
- removed R9: 4.7k, Resistor_SMD:R_0805_2012Metric_Pad1.20x1.40mm_HandSolder, symbol Device:R
- added C7: 1-5uF, Capacitor_SMD:C_0805_2012Metric_Pad1.18x1.45mm_HandSolder, symbol Device:C
- added C8: 0.1uF, Capacitor_SMD:C_0805_2012Metric_Pad1.18x1.45mm_HandSolder, symbol Device:C
- added J12: Conn_01x09_Pin, Connector_PinHeader_2.54mm:PinHeader_1x09_P2.54mm_Vertical, symbol Connector:Conn_01x09_Pin
- C5: value 10uF -> 1uF
- J1: footprint Connector_PinHeader_1.00mm:PinHeader_1x03_P1.00mm_Horizontal -> Connector_PinHeader_2.54mm:PinHeader_1x03_P2.54mm_Vertical
- J5, J7, J9: footprint Connector_PinHeader_2.54mm:PinHeader_1x03_P2.54mm_Horizontal -> Connector_PinHeader_2.54mm:PinHeader_1x03_P2.54mm_Vertical
Connections:
- net +3V3: no longer C5.1, U2.5 (VIO), U2.6 (VDD), U2.7 (REGIN)
- net GND: now also C7.2, C8.2; no longer C5.2
- net GPIO1: now also J12.1 (Pin_1)
- net GPIO19: now also J12.4 (Pin_4)
- net GPIO2: now also J12.2 (Pin_2)
- net GPIO20: now also J12.5 (Pin_5)
- net GPIO39: now also J12.6 (Pin_6)
- net GPIO40: now also J12.7 (Pin_7)
- net GPIO45: now also J12.8 (Pin_8)
- net GPIO48: now also J12.9 (Pin_9)
- net GPIO8: now also J12.3 (Pin_3)
- net at U2.9 (~{RST}): now also U2.5 (VIO), U2.6 (VDD), C7.1, C8.1
- new net: C5.2, U2.7 (REGIN)
- new net VBUS: C5.1
- no-connect marks 10 -> 11
Other:
- moved on the sheet: C6, U2
