File: moisture_sensor/moisture_sensor/moisture_sensor.kicad_pcb (KiCad board)
At the start: 2 copper layers, 9 parts, among them U1 LM358, U2 LM358

Commit message: V6
Parts:
- added J1: Conn_01x02_Socket, Connector_PinHeader_2.54mm:PinHeader_1x02_P2.54mm_Vertical, F.Cu at (122.0, 85.2)
- added J2: Moisture_Power, TerminalBlock_Phoenix:TerminalBlock_Phoenix_MKDS-1,5-2-5.08_1x02_P5.08mm_Horizontal, F.Cu at (123.5, 74.0)
- added J4: Conn_01x01_Pin, Connector_PinHeader_2.54mm:PinHeader_1x01_P2.54mm_Vertical, F.Cu at (122.0, 100.0)
- moved U2 10.6 mm to (145.3, 102.3)
- moved U1 7.60 mm to (145.3, 87.8)
- moved R1 1.51 mm to (130.0, 85.0)
- moved R2 1.46 mm to (130.0, 88.0)
- turned R7 to 180 degrees
Routing:
- net +3V3: track 0.00 -> 74.5 mm
- net Net-(U1B--): track 0.00 -> 32.4 mm, vias 0 -> 2
- net Net-(U2A-+): track 0.00 -> 27.5 mm
- net /Moisture_Sensor_Output: track 0.00 -> 26.7 mm, vias 0 -> 2
- net Net-(U1A--): track 0.00 -> 24.2 mm, vias 0 -> 2
- net Net-(U2A--): track 0.00 -> 21.3 mm
- net Net-(U1B-+): track 0.00 -> 19.8 mm
- net /Input_Probe_2: track 0.00 -> 7.10 mm
- net /Input_Probe_1: track 0.00 -> 7.09 mm
- net GND: track 0.00 -> 2.21 mm, vias 0 -> 1
- added copper zone on B.Cu, net GND
- added copper zone on F.Cu, net GND
Other:
- board outline added: 35.5 x 38.5 mm

Commit message: Final V7
Parts:
- added J3: Screw_Terminal_01x02, TerminalBlock_Phoenix:TerminalBlock_Phoenix_MKDS-1,5-2-5.08_1x02_P5.08mm_Horizontal, F.Cu at (152.8, 96.2)
Connections:
- U1 pad 4: GND -> -3V3
- U2 pad 4: GND -> -3V3
Routing:
- net -3V3: track 0.00 -> 33.1 mm
- net GND: track 2.21 -> 9.06 mm, vias 1 -> 3
Other:
- board size 35.5 x 38.5 mm -> 40.8 x 38.5 mm
